File: test1.brd (EAGLE design)
At the start: 42.9 x 55.9 mm, 14 parts, among them J1 POWER_JACK, J6 AVR_SPI_PROG_3X2NS, U2 328P

Commit message: s
s
Parts:
- moved R3 7.08 mm to (14.2, 11.4), turned to 270 degrees
Routing:
- net N$11: track 0.18 -> 15.8 mm
- net GND: track 129.5 -> 135.6 mm
- net N$3: track 0.00 -> 5.55 mm
Changed lines of the file:
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@@
 <setting verticaltext="up"/>
 </settings>
-<grid distance="0.05" unitdist="inch" unit="inch" style="lines" multiple="1" display="yes" altdistance="0.025" altunitdist="inch" altunit="inch"/>
+<grid distance="0.01" unitdist="inch" unit="inch" style="lines" multiple="1" display="yes" altdistance="0.025" altunitdist="inch" altunit="inch"/>
 <layers>
 <layer number="1" name="Top" color="4" fill="1" visible="yes" active="yes"/>
@@
 <text x="19.05" y="17.78" size="1.016" layer="121" rot="R90">0.1uF\</text>
 <text x="36.83" y="38.1" size="1.016" layer="121" rot="R90">0.1uF\</text>
+<text x="15.24" y="10.16" size="1.016" layer="121" rot="R90">10k</text>
 <text x="22.86" y="10.16" size="1.016" layer="121" rot="R90">10k</text>
 <text x="30.48" y="10.16" size="1.016" layer="121" rot="R90">10k</text>
@@
 <autorouter>
 <pass name="Default">
-<param name="RoutingGrid" value="50mil"/>
+<param name="RoutingGrid" value="12.5mil"/>
 <param name="AutoGrid" value="1"/>
 <param name="Efforts" value="0"/>
 <param name="TopRouterVariant" value="1"/>
 <param name="tpViaShape" value="round"/>
-<param name="PrefDir.1" value="a"/>
+<param name="PrefDir.1" value="-"/>
 <param name="PrefDir.2" value="0"/>
 <param name="PrefDir.3" value="0"/>
@@
 <param name="PrefDir.14" value="0"/>
 <param name="PrefDir.15" value="0"/>
-<param name="PrefDir.16" value="a"/>
+<param name="PrefDir.16" value="|"/>
 <param name="cfVia" value="8"/>
 <param name="cfNonPref" value="5"/>
@@
 <element name="R1" library="resistor" package="M3216" value="10K" x="27.94" y="11.43" rot="R90"/>
 <element name="R2" library="resistor" package="M3216" value="10K" x="20.32" y="11.43" rot="R90"/>
-<element name="R3" library="resistor" package="M3216" value="10K" x="7.62" y="13.97" rot="R90"/>
+<element name="R3" library="resistor" package="M3216" value="10K" x="14.224" y="11.43" rot="R270"/>
 <element name="R4" library="resistor" package="M3216" value="10K" x="34.29" y="34.29" rot="R90"/>
 <element name="U2" library="SparkFun-IC-Microcontroller" package="DIP28" value="328P" x="26.67" y="34.29" rot="R270">
@@
 <contactref element="J5" pad="6"/>
 <contactref element="J6" pad="6"/>
-<wire x1="20.3454" y1="13.0302" x2="20.3454" y2="14.1732" width="0.254" layer="1"/>
-<wire x1="20.3454" y1="14.1732" x2="20.3454" y2="18.288" width="0.254" layer="1"/>
-<wire x1="20.3454" y1="18.288" x2="20.32" y2="18.4" width="0.254" layer="1"/>
-<wire x1="20.3454" y1="13.0302" x2="20.32" y2="12.83" width="0.254" layer="1"/>
-<wire x1="12.573" y1="10.5156" x2="12.573" y2="10.0584" width="0" layer="19" extent="1-16"/>
-<wire x1="11.2014" y1="11.8872" x2="12.573" y2="10.5156" width="0" layer="19" extent="1-16"/>
-<wire x1="11.2014" y1="13.716" x2="11.2014" y2="11.8872" width="0" layer="19" extent="1-16"/>
-<wire x1="11.6586" y1="14.1732" x2="11.2014" y2="13.716" width="0" layer="19" extent="1-16"/>
-<wire x1="20.3454" y1="14.1732" x2="11.6586" y2="14.1732" width="0" layer="19" extent="1-16"/>
-<wire x1="12.573" y1="10.0584" x2="7.62" y2="12.57" width="0" layer="19" extent="1-16"/>
 <wire x1="20.3454" y1="12.8016" x2="27.8892" y2="12.8016" width="0.254" layer="1"/>
 <wire x1="27.8892" y1="12.8016" x2="27.94" y2="12.83" width="0.254" layer="1"/>
@@
 <wire x1="12.1158" y1="30.861" x2="11.97" y2="33.4" width="0.254" layer="16"/>
 <wire x1="22.86" y1="32.9184" x2="22.86" y2="33.02" width="0.254" layer="16"/>
+<wire x1="20.3454" y1="18.288" x2="20.3454" y2="13.0302" width="0.254" layer="1"/>
+<wire x1="20.3454" y1="13.0302" x2="20.32" y2="12.83" width="0.254" layer="1"/>
+<wire x1="20.3454" y1="18.288" x2="20.32" y2="18.4" width="0.254" layer="1"/>
+<wire x1="20.1168" y1="12.8016" x2="14.4018" y2="12.8016" width="0.254" layer="1"/>
+<wire x1="14.4018" y1="12.8016" x2="14.224" y2="12.83" width="0.254" layer="1"/>
+<wire x1="20.1168" y1="12.8016" x2="20.32" y2="12.83" width="0.254" layer="1"/>
 </signal>
 <signal name="N$3">
 <contactref element="R3" pad="2"/>
 <contactref element="LED3" pad="K"/>
-<wire x1="12.8016" y1="12.3444" x2="12.8016" y2="12.8016" width="0" layer="19" extent="1-16"/>
-<wire x1="14.1732" y1="10.9728" x2="12.8016" y2="12.3444" width="0" layer="19" extent="1-16"/>
-<wire x1="14.1732" y1="6.6294" x2="14.1732" y2="10.9728" width="0" layer="19" extent="1-16"/>
-<wire x1="12.8016" y1="5.2578" x2="14.1732" y2="6.6294" width="0" layer="19" extent="1-16"/>
-<wire x1="12.8016" y1="12.8016" x2="7.62" y2="15.37" width="0" layer="19" extent="1-16"/>
-<wire x1="12.8016" y1="5.2578" x2="12.7" y2="5.08" width="0" layer="19" extent="1-16"/>
+<wire x1="12.8016" y1="5.2578" x2="14.1732" y2="6.6294" width="0.254" layer="1"/>
+<wire x1="12.8016" y1="5.2578" x2="12.7" y2="5.08" width="0.254" layer="1"/>
+<wire x1="14.1732" y1="6.6294" x2="14.1732" y2="9.8298" width="0.254" layer="1"/>
+<wire x1="14.1732" y1="9.8298" x2="14.224" y2="10.03" width="0.254" layer="1"/>
 </signal>
 <signal name="N$4">
@@
 <contactref element="LED3" pad="A"/>
 <contactref element="U2" pad="14"/>
-<wire x1="15.3162" y1="10.0584" x2="15.3162" y2="5.2578" width="0" layer="19" extent="1-16"/>
-<wire x1="22.86" y1="17.6022" x2="15.3162" y2="10.0584" width="0" layer="19" extent="1-16"/>
-<wire x1="15.3162" y1="5.2578" x2="15.24" y2="5.08" width="0" layer="19" extent="1-16"/>
+<wire x1="15.3162" y1="10.0584" x2="15.3162" y2="5.2578" width="0.254" layer="16"/>
+<wire x1="22.86" y1="17.6022" x2="15.3162" y2="10.0584" width="0.254" layer="16"/>
+<wire x1="15.3162" y1="5.2578" x2="15.24" y2="5.08" width="0.254" layer="16"/>
 <wire x1="22.86" y1="17.6022" x2="22.86" y2="17.78" width="0.254" layer="16"/>
 </signal>
